File: KiCad/tiny_blinky/Tiny_Blinky_Power.sch (KiCad schematic (older format))
At the start: 6 parts, among them J3 Vin, J4 5V, U2 AP1117-50

Commit message: Session 2 updates
Parts:
- J3, J4: footprint Connector_PinHeader_2.54mm:PinHeader_1x02_P2.54mm_Vertical -> Connector_PinSocket_2.54mm:PinSocket_1x02_P2.54mm_Vertical
Changed lines of the file:
@@
 F 0 "J3" H 2650 3550 50  0000 C CNN
 F 1 "Vin" H 2650 3450 50  0000 C CNN
-F 2 "Connector_PinHeader_2.54mm:PinHeader_1x02_P2.54mm_Vertical" H 2525 3325 50  0001 C CNN
+F 2 "Connector_PinSocket_2.54mm:PinSocket_1x02_P2.54mm_Vertical" H 2525 3325 50  0001 C CNN
 F 3 "~" H 2525 3325 50  0001 C CNN
 	1    2525 3325
@@
 F 0 "J4" H 6050 3400 50  0000 L CNN
 F 1 "5V" H 6050 3300 50  0000 L CNN
-F 2 "Connector_PinHeader_2.54mm:PinHeader_1x02_P2.54mm_Vertical" H 6000 3375 50  0001 C CNN
+F 2 "Connector_PinSocket_2.54mm:PinSocket_1x02_P2.54mm_Vertical" H 6000 3375 50  0001 C CNN
 F 3 "~" H 6000 3375 50  0001 C CNN
 	1    6000 3375

Commit message: Session 3 & 4 updates
Parts:
- BT1: footprint Battery:BatteryHolder_Keystone_3002_1x2032 -> tiny_blinky:BatteryHolder_Keystone_3024-2x2032
- C1: footprint Capacitor_THT:CP_Radial_D8.0mm_P3.50mm -> tiny_blinky:CP_Radial_D8.0mm_P3.50mm
- C2: footprint Capacitor_THT:C_Disc_D5.0mm_W2.5mm_P2.50mm -> tiny_blinky:C_Disc_D5.0mm_W2.5mm_P2.50mm
- J3, J4: footprint Connector_PinSocket_2.54mm:PinSocket_1x02_P2.54mm_Vertical -> tiny_blinky:PinSocket_1x02_P2.54mm_Vertical
- U2: footprint Package_TO_SOT_SMD:SOT-223-3_TabPin2 -> tiny_blinky:SOT-223-3_TabPin2
Changed lines of the file:
@@
 $Descr A4 11693 8268
 encoding utf-8
-Sheet 2 2
+Sheet 2 3
 Title ""
 Date ""
@@
 F 0 "J3" H 2650 3550 50  0000 C CNN
 F 1 "Vin" H 2650 3450 50  0000 C CNN
-F 2 "Connector_PinSocket_2.54mm:PinSocket_1x02_P2.54mm_Vertical" H 2525 3325 50  0001 C CNN
+F 2 "tiny_blinky:PinSocket_1x02_P2.54mm_Vertical" H 2525 3325 50  0001 C CNN
 F 3 "~" H 2525 3325 50  0001 C CNN
 	1    2525 3325
@@
 F 0 "BT1" H 3175 3550 50  0000 L CNN
 F 1 "2xCR2032" H 3125 3375 50  0000 L CNN
-F 2 "Battery:BatteryHolder_Keystone_3002_1x2032" V 3100 3485 50  0001 C CNN
+F 2 "tiny_blinky:BatteryHolder_Keystone_3024-2x2032" V 3100 3485 50  0001 C CNN
 F 3 "~" V 3100 3485 50  0001 C CNN
 	1    3100 3425
@@
 F 0 "C1" H 3975 3475 50  0000 L CNN
 F 1 "470uF/25V" H 3975 3275 50  0000 L CNN
-F 2 "Capacitor_THT:CP_Radial_D8.0mm_P3.50mm" H 3988 3225 50  0001 C CNN
+F 2 "tiny_blinky:CP_Radial_D8.0mm_P3.50mm" H 3988 3225 50  0001 C CNN
 F 3 "~" H 3950 3375 50  0001 C CNN
 	1    3950 3375
@@
 F 0 "C2" H 5125 3475 50  0000 L CNN
 F 1 "100n" H 5125 3275 50  0000 L CNN
-F 2 "Capacitor_THT:C_Disc_D5.0mm_W2.5mm_P2.50mm" H 5138 3225 50  0001 C CNN
+F 2 "tiny_blinky:C_Disc_D5.0mm_W2.5mm_P2.50mm" H 5138 3225 50  0001 C CNN
 F 3 "~" H 5100 3375 50  0001 C CNN
 	1    5100 3375
@@
 F 0 "J4" H 6050 3400 50  0000 L CNN
 F 1 "5V" H 6050 3300 50  0000 L CNN
-F 2 "Connector_PinSocket_2.54mm:PinSocket_1x02_P2.54mm_Vertical" H 6000 3375 50  0001 C CNN
+F 2 "tiny_blinky:PinSocket_1x02_P2.54mm_Vertical" H 6000 3375 50  0001 C CNN
 F 3 "~" H 6000 3375 50  0001 C CNN
 	1    6000 3375
@@
 F 0 "U2" H 4575 3275 50  0000 C CNN
 F 1 "AP1117-50" H 4575 3175 50  0000 C CNN
-F 2 "Package_TO_SOT_SMD:SOT-223-3_TabPin2" H 4550 3200 50  0001 C CNN
+F 2 "tiny_blinky:SOT-223-3_TabPin2" H 4550 3200 50  0001 C CNN
 F 3 "http://www.diodes.com/datasheets/AP1117.pdf" H 4650 2750 50  0001 C CNN
 	1    4550 3000
