File: KiCad/tiny_blinky/tiny_blinky.kicad_pcb (KiCad board)
At the start: 2 copper layers, 71.1 x 40.6 mm, 21 parts, among them J1 Dout, J2 SPI, J3 Vin, J4 5V, SW1 SW, U1 ATtiny85-20PU, U2 AP1117-50

Commit message: Session 3 & 4 updates
Parts:
- BT1: footprint Battery:BatteryHolder_Keystone_3002_1x2032 -> tiny_blinky:BatteryHolder_Keystone_3024-2x2032
- C1: footprint Capacitor_THT:CP_Radial_D8.0mm_P3.50mm -> tiny_blinky:CP_Radial_D8.0mm_P3.50mm
- C2: footprint Capacitor_THT:C_Disc_D5.0mm_W2.5mm_P2.50mm -> tiny_blinky:C_Disc_D5.0mm_W2.5mm_P2.50mm
- D1, D2, D3: footprint LED_SMD:LED_WS2812B_PLCC4_5.0x5.0mm_P3.2mm -> tiny_blinky:LED_WS2812B_PLCC4_5.0x5.0mm_P3.2mm
- H1, H2, H3, H4: footprint MountingHole:MountingHole_3.2mm_M3_Pad_Via -> tiny_blinky:MountingHole_3.2mm_M3_Pad_Via
- J1: footprint Connector_PinSocket_2.54mm:PinSocket_1x03_P2.54mm_Vertical -> tiny_blinky:PinSocket_1x03_P2.54mm_Vertical
- J2: footprint Connector_PinHeader_2.54mm:PinHeader_2x03_P2.54mm_Vertical -> tiny_blinky:PinHeader_2x03_P2.54mm_Vertical
- J3, J4: footprint Connector_PinSocket_2.54mm:PinSocket_1x02_P2.54mm_Vertical -> tiny_blinky:PinSocket_1x02_P2.54mm_Vertical
- R1, R2: footprint Resistor_THT:R_Axial_DIN0207_L6.3mm_D2.5mm_P7.62mm_Horizontal -> tiny_blinky:R_Axial_DIN0207_L6.3mm_D2.5mm_P7.62mm_Horizontal
- SW1: footprint Button_Switch_THT:SW_PUSH_6mm_H5mm -> tiny_blinky:SW_PUSH_6mm_H5mm
- U1: footprint Package_DIP:DIP-8_W7.62mm -> tiny_blinky:DIP-8_W7.62mm
- U2: footprint Package_TO_SOT_SMD:SOT-223-3_TabPin2 -> tiny_blinky:SOT-223-3_TabPin2
- moved SW1 7.55 mm to (70.6, 34.0), turned to 270 degrees
- moved G2 7.37 mm to (66.5, 43.4)
- moved G1 4.32 mm to (101.6, 54.6)
Routing:
- net GND: track 191.9 -> 287.2 mm
- net /Tiny_Blinky_Power/Vin: track 65.6 -> 74.6 mm
- net /5V: track 124.5 -> 119.7 mm
- net Net-(R2-Pad1): track 28.8 -> 28.2 mm
- added copper zone on F.Cu, net /5V
Other:
- outline, holes or cut-outs redrawn
