File: KiCad/tiny_blinky/tiny_blinky.sch (KiCad schematic (older format))
At the start: 15 parts, among them J1 Dout, J2 SPI, SW1 SW, U1 ATtiny85-20PU

Commit message: Session 2 updates
Parts:
- removed G1: LOGO_skull_n_wrenches, tiny_blinky_v1:skull_n_wrenches, symbol tiny_blinky:LOGO_skull_n_wrenches
- removed H5: MountingHole_Pad, MountingHole:MountingHole_3.2mm_M3_Pad_Via, symbol Mechanical:MountingHole_Pad
- added G1: LOGO_skull, tiny_blinky:logo_skull, symbol tiny_blinky:LOGO_skull
- added H1: MountingHole_Pad, MountingHole:MountingHole_3.2mm_M3_Pad_Via, symbol Mechanical:MountingHole_Pad
- G2: footprint tiny_blinky_v1:hackaday -> tiny_blinky:logo_hackaday
Connections:
- net GND: now also H1.1
- net A0 renamed PB0
- net A1 renamed PB1
- net A2 renamed PB2
- net A3 renamed PB5
- net ADR0 renamed PGM0
- net ADR1 renamed PGM1
- net ADR2 renamed PGM2
- net ADR3 renamed PGM5
Other:
- note removed: "MECH AND VIRTUAL PARTS"
Changed lines of the file:
@@
 	2750 3700 3000 3700
 Text Label 3000 3200 2    50   ~ 0
-A0
+PB0
 Text Label 3000 3300 2    50   ~ 0
-A1
+PB1
 Text Label 3000 3400 2    50   ~ 0
-A2
+PB2
 Text Label 3000 3700 2    50   ~ 0
-A3
+PB5
 $Comp
 L tiny_blinky:Conn_02x03_Odd_Even J2
@@
 	4250 6675 3975 6675
 Text Label 3200 6475 0    50   ~ 0
-ADR1
+PGM1
 Text Label 3200 6575 0    50   ~ 0
-ADR2
+PGM2
 Text Label 3200 6675 0    50   ~ 0
-ADR3
+PGM5
 Text Label 4250 6575 2    50   ~ 0
-ADR0
+PGM0
 Text Label 4250 6675 2    50   ~ 0
 GND
@@
 	3100 6200 4350 6200
 Wire Notes Line
-	2900 5900 4600 5900
+	2650 5900 4600 5900
 Wire Notes Line
 	4600 5900 4600 6900
 Wire Notes Line
-	4600 6900 2900 6900
-Wire Notes Line
-	2900 6900 2900 5900
+	4600 6900 2650 6900
+Wire Notes Line
+	2650 6900 2650 5900
 Text Notes 4175 5975 2    50   ~ 10
 SPI PROGRAM HEADER
@@
 Wire Bus Line
 	4350 6475 4350 6200
-Text Label 3100 3100 0    50   ~ 0
-A[0..3]
-Text Label 4350 6200 2    50   ~ 0
-ADR[0..3]
+Text Label 3100 3925 2    50   ~ 0
+PB[0..5]
+Text Label 3100 6100 2    50   ~ 0
+PGM[0..5]
+$Comp
+L Mechanical:MountingHole_Pad H1
+U 1 1 5F070680
+P 7075 5350
+F 0 "H1" H 7200 5400 50  0000 L CNN
+F 1 "MountingHole_Pad" H 7200 5325 50  0001 L CNN
+F 2 "MountingHole:MountingHole_3.2mm_M3_Pad_Via" H 7075 5350 50  0001 C CNN
+F 3 "~" H 7075 5350 50  0001 C CNN
+	1    7075 5350
+	1    0    0    -1
+$EndComp
+$Comp
+L power:GND #PWR04
+U 1 1 5F070B68
+P 7075 5450
+F 0 "#PWR04" H 7075 5200 50  0001 C CNN
+F 1 "GND" H 7125 5250 50  0000 C CNN
+F 2 "" H 7075 5450 50  0001 C CNN
+F 3 "" H 7075 5450 50  0001 C CNN
+	1    7075 5450
+	1    0    0    -1
+$EndComp
 $Comp
 L Mechanical:MountingHole_Pad H2
-U 1 1 5EFED2BD
-P 6975 5775
-F 0 "H2" H 7100 5800 50  0000 L CNN
-F 1 "MountingHole_Pad" H 7100 5775 50  0001 L CNN
-F 2 "MountingHole:MountingHole_3.2mm_M3_Pad_Via" H 6975 5775 50  0001 C CNN
-F 3 "~" H 6975 5775 50  0001 C CNN
-	1    6975 5775
+U 1 1 5F070F04
+P 7450 5350
+F 0 "H2" H 7575 5400 50  0000 L CNN
+F 1 "MountingHole_Pad" H 7575 5325 50  0001 L CNN
+F 2 "MountingHole:MountingHole_3.2mm_M3_Pad_Via" H 7450 5350 50  0001 C CNN
+F 3 "~" H 7450 5350 50  0001 C CNN
+	1    7450 5350
+	1    0    0    -1
+$EndComp
+$Comp
+L power:GND #PWR05
+U 1 1 5F070F0E
+P 7450 5450
+F 0 "#PWR05" H 7450 5200 50  0001 C CNN
+F 1 "GND" H 7500 5250 50  0000 C CNN
+F 2 "" H 7450 5450 50  0001 C CNN
+F 3 "" H 7450 5450 50  0001 C CNN
+	1    7450 5450
 	1    0    0    -1
 $EndComp
 $Comp
 L Mechanical:MountingHole_Pad H3
-U 1 1 5EFED427
-P 7475 5775
-F 0 "H3" H 7600 5800 50  0000 L CNN
-F 1 "MountingHole_Pad" H 7600 5775 50  0001 L CNN
-F 2 "MountingHole:MountingHole_3.2mm_M3_Pad_Via" H 7475 5775 50  0001 C CNN
-F 3 "~" H 7475 5775 50  0001 C CNN
-	1    7475 5775
+U 1 1 5F072039
+P 7825 5350
+F 0 "H3" H 7950 5400 50  0000 L CNN
+F 1 "MountingHole_Pad" H 7950 5325 50  0001 L CNN
+F 2 "MountingHole:MountingHole_3.2mm_M3_Pad_Via" H 7825 5350 50  0001 C CNN
+F 3 "~" H 7825 5350 50  0001 C CNN
+	1    7825 5350
+	1    0    0    -1
+$EndComp
+$Comp
+L power:GND #PWR06
+U 1 1 5F072043
+P 7825 5450
+F 0 "#PWR06" H 7825 5200 50  0001 C CNN
+F 1 "GND" H 7875 5250 50  0000 C CNN
+F 2 "" H 7825 5450 50  0001 C CNN
+F 3 "" H 7825 5450 50  0001 C CNN
+	1    7825 5450
 	1    0    0    -1
 $EndComp
 $Comp
 L Mechanical:MountingHole_Pad H4
-U 1 1 5EFED77D
-P 7975 5775
-F 0 "H4" H 8100 5800 50  0000 L CNN
-F 1 "MountingHole_Pad" H 8100 5775 50  0001 L CNN
-F 2 "MountingHole:MountingHole_3.2mm_M3_Pad_Via" H 7975 5775 50  0001 C CNN
-F 3 "~" H 7975 5775 50  0001 C CNN
-	1    7975 5775
-	1    0    0    -1
-$EndComp
-$Comp
-L Mechanical:MountingHole_Pad H5
-U 1 1 5EFEDA5C
-P 8475 5775
-F 0 "H5" H 8600 5800 50  0000 L CNN
-F 1 "MountingHole_Pad" H 8600 5775 50  0001 L CNN
-F 2 "MountingHole:MountingHole_3.2mm_M3_Pad_Via" H 8475 5775 50  0001 C CNN
-F 3 "~" H 8475 5775 50  0001 C CNN
-	1    8475 5775
-	1    0    0    -1
-$EndComp
-Wire Wire Line
-	6975 5875 6975 6100
-Wire Wire Line
-	6975 6100 7475 6100
-Wire Wire Line
-	8475 6100 8475 5875
-Wire Wire Line
-	7975 5875 7975 6100
-Connection ~ 7975 6100
-Wire Wire Line
-	7975 6100 8475 6100
-Wire Wire Line
-	7475 5875 7475 6100
-Connection ~ 7475 6100
-Wire Wire Line
-	7475 6100 7975 6100
-Text Label 6975 6100 0    50   ~ 0
-GND
-Text Notes 6975 5525 0    50   ~ 10
-MECH AND VIRTUAL PARTS
+U 1 1 5F07204D
+P 8200 5350
+F 0 "H4" H 8325 5400 50  0000 L CNN
+F 1 "MountingHole_Pad" H 8325 5325 50  0001 L CNN
+F 2 "MountingHole:MountingHole_3.2mm_M3_Pad_Via" H 8200 5350 50  0001 C CNN
+F 3 "~" H 8200 5350 50  0001 C CNN
+	1    8200 5350
+	1    0    0    -1
+$EndComp
+$Comp
+L power:GND #PWR07
+U 1 1 5F072057
+P 8200 5450
+F 0 "#PWR07" H 8200 5200 50  0001 C CNN
+F 1 "GND" H 8250 5250 50  0000 C CNN
+F 2 "" H 8200 5450 50  0001 C CNN
+F 3 "" H 8200 5450 50  0001 C CNN
+	1    8200 5450
+	1    0    0    -1
+$EndComp
+$Comp
+L tiny_blinky:LOGO_hackaday G2
+U 1 1 5F0752BD
+P 10175 6725
+F 0 "G2" H 10175 7075 60  0001 C CNN
+F 1 "LOGO_hackaday" H 10175 6950 60  0001 C CNN
+F 2 "tiny_blinky:logo_hackaday" H 10175 6725 50  0001 C CNN
+F 3 "" H 10175 6725 50  0001 C CNN
+	1    10175 6725
+	1    0    0    -1
+$EndComp
+$Comp
+L tiny_blinky:LOGO_skull G1
+U 1 1 5F075902
+P 10750 6075
+F 0 "G1" H 10750 5761 60  0001 C CNN
+F 1 "LOGO_skull" H 10750 6389 60  0001 C CNN
+F 2 "tiny_blinky:logo_skull" H 10750 6075 50  0001 C CNN
+F 3 "" H 10750 6075 50  0001 C CNN
+	1    10750 6075
+	1    0    0    -1
+$EndComp
 Wire Bus Line
 	3100 6200 3100 6575
 Wire Bus Line
 	3100 3100 3100 6200
-$Comp
-L tiny_blinky:LOGO_hackaday G2
-U 1 1 5EFF6A43
-P 10750 7050
-F 0 "G2" H 10750 7022 60  0001 C CNN
-F 1 "LOGO_hackaday" H 10750 7078 60  0001 C CNN
-F 2 "tiny_blinky_v1:hackaday" H 10750 7050 50  0001 C CNN
-F 3 "" H 10750 7050 50  0001 C CNN
-	1    10750 7050
-	1    0    0    -1
-$EndComp
-$Comp
-L tiny_blinky:LOGO_skull_n_wrenches G1
-U 1 1 5EFF8990
-P 10950 6800
-F 0 "G1" H 10950 6664 60  0001 C CNN
-F 1 "LOGO_skull_n_wrenches" H 10950 6936 60  0001 C CNN
-F 2 "tiny_blinky_v1:skull_n_wrenches" H 10950 6800 50  0001 C CNN
-F 3 "" H 10950 6800 50  0001 C CNN
-	1    10950 6800
-	1    0    0    -1
-$EndComp
 $EndSCHEMATC

Commit message: Session 3 & 4 updates
Parts:
- D1, D2, D3: footprint LED_SMD:LED_WS2812B_PLCC4_5.0x5.0mm_P3.2mm -> tiny_blinky:LED_WS2812B_PLCC4_5.0x5.0mm_P3.2mm
- H1, H2, H3, H4: footprint MountingHole:MountingHole_3.2mm_M3_Pad_Via -> tiny_blinky:MountingHole_3.2mm_M3_Pad_Via
- J1: footprint Connector_PinSocket_2.54mm:PinSocket_1x03_P2.54mm_Vertical -> tiny_blinky:PinSocket_1x03_P2.54mm_Vertical
- J2: footprint Connector_PinHeader_2.54mm:PinHeader_2x03_P2.54mm_Vertical -> tiny_blinky:PinHeader_2x03_P2.54mm_Vertical
- R1, R2: footprint Resistor_THT:R_Axial_DIN0207_L6.3mm_D2.5mm_P7.62mm_Horizontal -> tiny_blinky:R_Axial_DIN0207_L6.3mm_D2.5mm_P7.62mm_Horizontal
- SW1: footprint Button_Switch_THT:SW_PUSH_6mm_H5mm -> tiny_blinky:SW_PUSH_6mm_H5mm
- U1: footprint Package_DIP:DIP-8_W7.62mm -> tiny_blinky:DIP-8_W7.62mm
Changed lines of the file:
@@
 $Descr A4 11693 8268
 encoding utf-8
-Sheet 1 2
+Sheet 1 3
 Title "TINY_BLINKY"
 Date "2020-06-27"
@@
 F 0 "U1" H 1750 4075 50  0000 R CNN
 F 1 "ATtiny85-20PU" V 1725 3800 50  0000 R CNN
-F 2 "Package_DIP:DIP-8_W7.62mm" H 2150 3500 50  0001 C CIN
+F 2 "tiny_blinky:DIP-8_W7.62mm" H 2150 3500 50  0001 C CIN
 F 3 "http://ww1.microchip.com/downloads/en/DeviceDoc/atmel-2586-avr-8-bit-microcontroller-attiny25-attiny45-attiny85_datasheet.pdf" H 2150 3500 50  0001 C CNN
 	1    2150 3500
 	1    0    0    -1
-$EndComp
-$Comp
-L tiny_blinky:SW_Push SW1
-U 1 1 5EF7BBA3
-P 3550 2575
-F 0 "SW1" V 3475 2725 50  0000 L CNN
-F 1 "SW" V 3575 2725 50  0000 L CNN
-F 2 "Button_Switch_THT:SW_PUSH_6mm_H5mm" H 3550 2775 50  0001 C CNN
-F 3 "~" H 3550 2775 50  0001 C CNN
-	1    3550 2575
-	0    1    1    0
 $EndComp
 $Comp
@@
 F 0 "R2" V 3550 4200 50  0000 L CNN
 F 1 "10k" V 3650 4225 50  0000 L CNN
-F 2 "Resistor_THT:R_Axial_DIN0207_L6.3mm_D2.5mm_P7.62mm_Horizontal" V 3480 4250 50  0001 C CNN
+F 2 "tiny_blinky:R_Axial_DIN0207_L6.3mm_D2.5mm_P7.62mm_Horizontal" V 3480 4250 50  0001 C CNN
 F 3 "~" H 3550 4250 50  0001 C CNN
 	1    3550 4250
@@
 F 0 "R1" V 4300 3600 50  0000 C CNN
 F 1 "330E" V 4350 3800 50  0000 C CNN
-F 2 "Resistor_THT:R_Axial_DIN0207_L6.3mm_D2.5mm_P7.62mm_Horizontal" V 4230 3600 50  0001 C CNN
+F 2 "tiny_blinky:R_Axial_DIN0207_L6.3mm_D2.5mm_P7.62mm_Horizontal" V 4230 3600 50  0001 C CNN
 F 3 "~" H 4300 3600 50  0001 C CNN
 	1    4300 3600
@@
 F 0 "D1" H 6150 3850 50  0000 L CNN
 F 1 "WS2812B" H 6250 3775 50  0000 L CNN
-F 2 "LED_SMD:LED_WS2812B_PLCC4_5.0x5.0mm_P3.2mm" H 6075 3300 50  0001 L TNN
+F 2 "tiny_blinky:LED_WS2812B_PLCC4_5.0x5.0mm_P3.2mm" H 6075 3300 50  0001 L TNN
 F 3 "https://cdn-shop.adafruit.com/datasheets/WS2812B.pdf" H 6125 3225 50  0001 L TNN
 	1    6025 3600
@@
 F 0 "D2" H 7650 3850 50  0000 L CNN
 F 1 "WS2812B" H 7750 3775 50  0000 L CNN
-F 2 "LED_SMD:LED_WS2812B_PLCC4_5.0x5.0mm_P3.2mm" H 7575 3300 50  0001 L TNN
+F 2 "tiny_blinky:LED_WS2812B_PLCC4_5.0x5.0mm_P3.2mm" H 7575 3300 50  0001 L TNN
 F 3 "https://cdn-shop.adafruit.com/datasheets/WS2812B.pdf" H 7625 3225 50  0001 L TNN
 	1    7525 3600
@@
 F 0 "D3" H 9150 3850 50  0000 L CNN
 F 1 "WS2812B" H 9250 3775 50  0000 L CNN
-F 2 "LED_SMD:LED_WS2812B_PLCC4_5.0x5.0mm_P3.2mm" H 9075 3300 50  0001 L TNN
+F 2 "tiny_blinky:LED_WS2812B_PLCC4_5.0x5.0mm_P3.2mm" H 9075 3300 50  0001 L TNN
 F 3 "https://cdn-shop.adafruit.com/datasheets/WS2812B.pdf" H 9125 3225 50  0001 L TNN
 	1    9025 3600
@@
 F 0 "J1" H 10300 3650 50  0000 L CNN
 F 1 "Dout" H 10300 3550 50  0000 L CNN
-F 2 "Connector_PinSocket_2.54mm:PinSocket_1x03_P2.54mm_Vertical" H 10250 3600 50  0001 C CNN
+F 2 "tiny_blinky:PinSocket_1x03_P2.54mm_Vertical" H 10250 3600 50  0001 C CNN
 F 3 "~" H 10250 3600 50  0001 C CNN
 	1    10250 3600
@@
 F 0 "J2" H 3725 6850 50  0000 C CNN
 F 1 "SPI" H 3725 6775 50  0000 C CNN
-F 2 "Connector_PinHeader_2.54mm:PinHeader_2x03_P2.54mm_Vertical" H 3675 6575 50  0001 C CNN
+F 2 "tiny_blinky:PinHeader_2x03_P2.54mm_Vertical" H 3675 6575 50  0001 C CNN
 F 3 "~" H 3675 6575 50  0001 C CNN
 	1    3675 6575
@@
 F 0 "H1" H 7200 5400 50  0000 L CNN
 F 1 "MountingHole_Pad" H 7200 5325 50  0001 L CNN
-F 2 "MountingHole:MountingHole_3.2mm_M3_Pad_Via" H 7075 5350 50  0001 C CNN
+F 2 "tiny_blinky:MountingHole_3.2mm_M3_Pad_Via" H 7075 5350 50  0001 C CNN
 F 3 "~" H 7075 5350 50  0001 C CNN
 	1    7075 5350
@@
 F 0 "H2" H 7575 5400 50  0000 L CNN
 F 1 "MountingHole_Pad" H 7575 5325 50  0001 L CNN
-F 2 "MountingHole:MountingHole_3.2mm_M3_Pad_Via" H 7450 5350 50  0001 C CNN
+F 2 "tiny_blinky:MountingHole_3.2mm_M3_Pad_Via" H 7450 5350 50  0001 C CNN
 F 3 "~" H 7450 5350 50  0001 C CNN
 	1    7450 5350
@@
 F 0 "H3" H 7950 5400 50  0000 L CNN
 F 1 "MountingHole_Pad" H 7950 5325 50  0001 L CNN
-F 2 "MountingHole:MountingHole_3.2mm_M3_Pad_Via" H 7825 5350 50  0001 C CNN
+F 2 "tiny_blinky:MountingHole_3.2mm_M3_Pad_Via" H 7825 5350 50  0001 C CNN
 F 3 "~" H 7825 5350 50  0001 C CNN
 	1    7825 5350
@@
 F 0 "H4" H 8325 5400 50  0000 L CNN
 F 1 "MountingHole_Pad" H 8325 5325 50  0001 L CNN
-F 2 "MountingHole:MountingHole_3.2mm_M3_Pad_Via" H 8200 5350 50  0001 C CNN
+F 2 "tiny_blinky:MountingHole_3.2mm_M3_Pad_Via" H 8200 5350 50  0001 C CNN
 F 3 "~" H 8200 5350 50  0001 C CNN
 	1    8200 5350
@@
 	1    0    0    -1
 $EndComp
+$Sheet
+S 9550 1025 1275 950
+U 5F10C232
+F0 "routing" 50
+F1 "routing.sch" 50
+$EndSheet
+$Comp
+L tiny_blinky:SW_Push SW1
+U 1 1 5F1CB5ED
+P 3550 2575
+F 0 "SW1" V 3475 2800 50  0000 L CNN
+F 1 "SW" V 3575 2800 50  0000 L CNN
+F 2 "tiny_blinky:SW_PUSH_6mm_H5mm" H 3550 2775 50  0001 C CNN
+F 3 "" H 3550 2775 50  0001 C CNN
+	1    3550 2575
+	0    1    1    0
+$EndComp
 Wire Bus Line
